File: laptop-mainboard/kicad/07_ethernet.kicad_sch (KiCad schematic)
At the start: 8 parts, among them U34 RTL8125BG, U35 RTL8125BG, Y3 XTAL_25M, Y4 XTAL_25M

Commit message: Rev B: echte AM5-Pinbelegung, Kleinteile, EliteBook-850-G7-Format
- AM5-Pinmap (1718 Pins, WikiChip/Wikimedia Public Domain) als CSV,
  Sockel-Footprint mit echten Padnamen und 1708 Signal-Netzen im Board
- Blatt 10: MLCC-Baenke, 11 ESD-Arrays, USB2-Chokes, Straps; 48-MHz-Quarz;
  beidseitige Bestueckung (B.Cu) mit Kollisionspruefung pro Seite
- Board 340x112mm im EliteBook-850-G7-Layout: USB-C-100W-PD an der
  Barrel-Jack-Position, TB4/HDMI/USB-A/RJ45 rechts, USB-A/Klinke links,
  HP-Akku 3S/56Wh, HP-FPC-Steckplaetze (Pinouts zu verifizieren)
- GND-Stitching-Vias, MDI-/DP-Korridore, 645 Board-Netze
- Renderer tools/render_board.py erzeugt docs/board_render.png
- Doku: elitebook.md neu, grenzen.md/README/power/layout aktualisiert

Co-Authored-By: Claude Fable 5 <noreply@anthropic.com>
Claude-Session: https://claude.ai/code/session_01E8mU1RUAv938Hs69waADCc
Parts:
- removed C14: C_1n_2kV, laptop_mainboard:C_1812, symbol lm:C_1n_2kV_C14
- removed J_LAN2: RJ45_Magjack_2G5, laptop_mainboard:RJ45_MAGJACK, symbol lm:RJ45_Magjack_2G5_J_LAN2
- removed U35: RTL8125BG, laptop_mainboard:QFN48_6x6, symbol lm:RTL8125BG_U35
- removed Y4: XTAL_25M, laptop_mainboard:XTAL_3225, symbol lm:XTAL_25M_Y4
Other:
- note added: "RJ45 rechts vorn wie beim EliteBook 850 G7 (Klappmechanik-Buchse)."
- note added: "Realtek RTL8125BG an SoC-GPP-Lane G0 (PCIe Gen2 x1)."
- note added: "Wake-on-LAN ueber PE_WAKE# (Open-Drain)."
- note removed: "2x Realtek RTL8125BG an SoC-GPP-Lanes G0/G1 (PCIe Gen2 x1)."
- note removed: "Wake-on-LAN ueber PE_WAKE# (gemeinsame Open-Drain-Leitung)."
- title: 2x 2.5-Gigabit-Ethernet -> 2.5-Gigabit-Ethernet
